File: apps/field/pcb/field_carrier.kicad_sch (KiCad schematic)
At the start: 5 parts, among them J1 XIAO_ESP32C6, J3 E220_EV2, J4 ログ_UART0

Commit message: feat(field): 台を EXPE7-4-6 に合わせて 55×45 で作り直し、表示の LED（D1〜D3・R1〜R6）を回路図と基板に足す
- 回路図: XIAO の D4・D5（920 の送信・受信）と D8・D9（2.4 の送信・受信）を 330 Ω 経由で
  D2・D3（OSRGHC3132A・赤＝送信・緑＝受信）へ。D1＝電源（5V から 1 kΩ×2・赤と黄緑で黄）。ERC 0 件
- 基板: 外形 55.0×45.0（切り欠きなし）。XIAO は基板の縁を y 45.5（受け口の面が背面パネルの外面と面一）。
  LED は背面の端（x 9.0・14.08・19.16・ランドの列 y 43.73）。抵抗は EV2 の下（EV2 は約 11 mm 浮く）に
  2.54 間隔＝LED の足から 7 ピンの隙間を真っすぐ通る。C1 は EV2 の 6・7 番の前、C2 は XIAO の右、J4 は右前
- 専用フットプリント: LED_D3.0mm-3_Horizontal_Staggered を足した（ランド 1.5＝背面端まで 0.5 を守る）。
  XIAO は受け口が縁から 2 mm 出る分を込み合いの枠に足し、シルクを台の上に収めた。EV2 の込み合いの枠は
  ソケットだけ（下に低い部品を置けるように）
- DRC（回路図との照合つき）＝違反 0・未配線 0・不一致 0

HARDWARE.md §3・§4 と wiring.svg はまだ直していない（次の作業）。

Co-Authored-By: Claude Opus 5.5 <noreply@anthropic.com>
Parts:
- added D1, D2, D3: OSRGHC3132A, field_carrier:LED_D3.0mm-3_Horizontal_Staggered, symbol Device:LED_Dual_AKA
- added R1, R2, R3, R4: 330, Resistor_THT:R_Axial_DIN0204_L3.6mm_D1.6mm_P5.08mm_Horizontal, symbol Device:R
- added R5, R6: 1k, Resistor_THT:R_Axial_DIN0204_L3.6mm_D1.6mm_P5.08mm_Horizontal, symbol Device:R
Connections:
- net +5V: now also R5.1, R6.1
- net GND: now also D1.2 (K), D2.2 (K), D3.2 (K)
- net LED24_RX: now reaches J1.10 (D9)
- net LED24_RX: now also R4.1
- net LED24_TX: now reaches J1.9 (D8)
- net LED24_TX: now also R3.1
- net LED920_TX: now reaches J1.5 (D4)
- net LED920_TX: now also R1.1
- net LED920_RX: now reaches J1.6 (D5)
- net LED920_RX: now also R2.1
- new net: D3.3 (A2), R4.2
- new net: D1.1 (A1), R5.2
- new net: D1.3 (A2), R6.2
- new net: D3.1 (A1), R3.2
- new net: D2.1 (A1), R1.2
- new net: D2.3 (A2), R2.2
- no-connect marks 5 -> 1
Other:
- note added: "D1＝電源（5V から常時・赤と黄緑を両方点ける＝黄）"
- note added: "D2＝920 MHz（送信＝赤・受信＝緑）"
- note added: "D3＝2.4 GHz（送信＝赤・受信＝緑）"
- note added: "Field の台（2 台同じ基板）＝XIAO と EV2 をピンソケットで差すだけ。高周波の線は引かない （2.4 GHz は XIAO の U.FL からピグテール・920 MHz は EV2 の SMA＝基準面は今のまま）。 結線の正典は apps/field/HARDWARE.md §3 と wiring.svg（直すときは同じコミットで）。 J1＝XIAO（表面を台へ向けて差す＝フットプリントは公式の鏡像・2 列は 15.24 mm）。 J3＝EV2（ユニット B＝SMA 寄りの GND スルーホール 3 つ＝支えのため・7 ピン列から 31.50 mm）。寸法は field_carrier.pretty の中で固定。 XIAO の 3V3 は使わない。D4・D5＝920 の送信・受信、D8・D9＝2.4 の送信・受信を表示の LED（D2・D3）へ。 D1〜D3＝OSRGHC3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"
- note removed: "Field の台（2 台同じ基板）＝XIAO と EV2 をピンソケットで差すだけ。高周波の線は引かない （2.4 GHz は XIAO の U.FL からピグテール・920 MHz は EV2 の SMA＝基準面は今のまま）。 結線の正典は apps/field/HARDWARE.md §3 と wiring.svg（直すときは同じコミットで）。 J1＝XIAO（表面を台へ向けて差す＝フットプリントは公式の鏡像・2 列は 15.24 mm）。 J3＝EV2（ユニット B＝SMA 寄りの GND スルーホール 3 つ＝支えのため・7 ピン列から 31.50 mm）。寸法は field_carrier.pretty の中で固定。 XIAO の 3V3・D4・D5・D8・D9 は使わない。"

Commit message: feat(field): 表示の LED を 1 列のフットプリントへ置き換え、アノードと EV2_RXD を引き直す
- 専用フットプリントを LED_D3.0mm-3_Horizontal_Staggered（三角）から
  LED_D3.0mm-3_Horizontal_O2.54mm_Z2.0mm（足 3 本を 2.54 間隔の 1 列）へ。
  曲げる位置はつばから 2.54＝データシートの樹脂のはみ出し（1.5MAX）と外側の足の開き
  （つばの下 約 1.1 で 2.54 に開き終わる）の両方から外れる。軸の高さ Z 2.0 とつばを
  背面パネルの内面に当てる位置は前のまま
- 配置: D3・D2・D1＝中心 x 8.45・15.25・22.05、ランドの列 y 42.46（6.8 間隔・ランド 1.5）。
  D3 の穴の縁 6.85 は穴あけ範囲（有効寸法 41.5）の左端 6.75 まで 0.1。外側のフレームの
  窓の縁（図面 p002 の正面図を画素で測った・LED の軸の高さで x 5.59）までは 約 1.26
- 裏: アノード 6 本は y 41.4 から 45° でそろえて寄せ、EV2 の 7 ピンの隙間を抜けて抵抗へ
  （抵抗の並びは前のまま）。表: EV2_RXD は XIAO の 1 番から斜めに下げ、LED のランドの前
  （y 40.93）を通って TXD の外を回る
- 新しい線に乗った GND の縫いビア 3 つを除いた（75 → 72）。XIAO の込み合いの枠は
  EV2 と同じくソケットの 2 列だけにした（モジュールは約 11 mm 浮く・LED は高さ 約 3.9）
- DRC（回路図との照合つき）＝違反 0・未配線 0・不一致 0。ERC 0

Co-Authored-By: Claude Opus 5.5 <noreply@anthropic.com>
Parts:
- D1, D2, D3: footprint field_carrier:LED_D3.0mm-3_Horizontal_Staggered -> field_carrier:LED_D3.0mm-3_Horizontal_O2.54mm_Z2.0mm
Changed lines of the file:
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@@
 			)
 		)
-		(property "Footprint" "field_carrier:LED_D3.0mm-3_Horizontal_Staggered"
+		(property "Footprint" "field_carrier:LED_D3.0mm-3_Horizontal_O2.54mm_Z2.0mm"
 			(at 38.1 175.26 0)
 			(hide yes)
@@
 			)
 		)
-		(property "Footprint" "field_carrier:LED_D3.0mm-3_Horizontal_Staggered"
+		(property "Footprint" "field_carrier:LED_D3.0mm-3_Horizontal_O2.54mm_Z2.0mm"
 			(at 88.9 175.26 0)
 			(hide yes)
@@
 			)
 		)
-		(property "Footprint" "field_carrier:LED_D3.0mm-3_Horizontal_Staggered"
+		(property "Footprint" "field_carrier:LED_D3.0mm-3_Horizontal_O2.54mm_Z2.0mm"
 			(at 139.7 175.26 0)
 			(hide yes)
